Commit message: updated urdf to work with pinocchio

File: franka_panda/panda.urdf (robot description, URDF)
Before this commit: robot panda, 13 links, 12 joints
Links:
- link panda_hand: geometry collision mesh filename=./franka_panda/meshes/collision/hand.obj; visual mesh filename=./franka_panda/meshes/visual/hand.obj
- link panda_leftfinger: geometry collision mesh filename=./franka_panda/meshes/collision/finger.obj; visual mesh filename=./franka_panda/meshes/visual/finger.obj
- link panda_link0: geometry collision mesh filename=./franka_panda/meshes/collision/link0.obj; visual mesh filename=./franka_panda/meshes/collision/link0.obj
- link panda_link1: geometry collision mesh filename=./franka_panda/meshes/collision/link1.obj; visual mesh filename=./franka_panda/meshes/visual/link1.obj
- link panda_link2: geometry collision mesh filename=./franka_panda/meshes/collision/link2.obj; visual mesh filename=./franka_panda/meshes/visual/link2.obj
- link panda_link3: geometry collision mesh filename=./franka_panda/meshes/collision/link3.obj; visual mesh filename=./franka_panda/meshes/visual/link3.obj
- link panda_link4: geometry collision mesh filename=./franka_panda/meshes/collision/link4.obj; visual mesh filename=./franka_panda/meshes/visual/link4.obj
- link panda_link5: geometry collision mesh filename=./franka_panda/meshes/collision/link5.obj; visual mesh filename=./franka_panda/meshes/visual/link5.obj
- link panda_link6: geometry collision mesh filename=./franka_panda/meshes/collision/link6.obj; visual mesh filename=./franka_panda/meshes/visual/link6.obj
- link panda_link7: geometry collision mesh filename=./franka_panda/meshes/collision/link7.obj; visual mesh filename=./franka_panda/meshes/collision/link7.obj
- link panda_rightfinger: geometry collision mesh filename=./franka_panda/meshes/collision/finger.obj; visual mesh filename=./franka_panda/meshes/visual/finger.obj
